Commit message: feat(phase5): add verified vision-driven pick and place runtime

File: ros2_ws/src/abb_lab_gripper/urdf/irb1200_5_90_gz_gripper_control.urdf.xacro (robot description, xacro)
@@ -3,4 +3,8 @@
   <xacro:arg name="prefix" default=""/>
   <xacro:arg name="controller_config_file" default="$(find abb_lab_gripper)/config/irb1200_gripper_controllers.yaml"/>
+  <xacro:arg name="world_to_base_z" default="0"/>
+  <!-- Keep the P3/P4 zero pose as the default.  Phase 5 passes a separate,
+       collision-free initial-state file through its isolated launch path. -->
+  <xacro:arg name="arm_initial_positions_file" default="$(find abb_lab_gripper)/config/arm_initial_positions.yaml"/>
   <!-- This wrapper deliberately reuses only the pinned ABB geometry macro.
        It does not include the existing arm-only control profile. -->
@@ -10,10 +14,12 @@
   <xacro:property name="prefix" value="$(arg prefix)"/>
   <xacro:property name="controller_config_file" value="$(arg controller_config_file)"/>
+  <xacro:property name="world_to_base_z" value="$(arg world_to_base_z)"/>
   <xacro:property name="arm_joint_limits" value="${xacro.load_yaml('$(find abb_lab_description)/config/irb1200_5_90_control_limits.yaml')['joint_limits']}"/>
   <xacro:property name="gripper_joint_limits" value="${xacro.load_yaml('$(find abb_lab_gripper)/config/two_finger_gripper_limits.yaml')['joint_limits']}"/>
   <xacro:property name="gripper_initial_positions" value="${xacro.load_yaml('$(find abb_lab_gripper)/config/two_finger_gripper_limits.yaml')['initial_positions']}"/>
+  <xacro:property name="arm_initial_positions" value="${xacro.load_yaml('$(arg arm_initial_positions_file)')['initial_positions']}"/>
   <link name="world"/>
   <joint name="${prefix}world_to_base" type="fixed">
-    <origin xyz="0 0 0" rpy="0 0 0"/>
+    <origin xyz="0 0 ${world_to_base_z}" rpy="0 0 0"/>
     <parent link="world"/>
     <child link="${prefix}base_link"/>
@@ -28,4 +34,5 @@
     prefix="${prefix}"
     arm_joint_limits="${arm_joint_limits}"
+    arm_initial_positions="${arm_initial_positions}"
     gripper_joint_limits="${gripper_joint_limits}"
     gripper_initial_positions="${gripper_initial_positions}"/>

File: ros2_ws/src/abb_lab_gripper/urdf/irb1200_5_90_gz_gripper_ros2_control.xacro (robot description, xacro)
@@ -4,5 +4,5 @@
        gripper finger exports state only: it is a URDF mimic follower, not a
        second command target. -->
-  <xacro:macro name="abb_irb1200_5_90_gz_gripper_ros2_control" params="name prefix arm_joint_limits gripper_joint_limits gripper_initial_positions">
+  <xacro:macro name="abb_irb1200_5_90_gz_gripper_ros2_control" params="name prefix arm_joint_limits arm_initial_positions gripper_joint_limits gripper_initial_positions">
     <ros2_control name="${name}" type="system">
       <hardware>
@@ -14,5 +14,7 @@
           <param name="max">${arm_joint_limits['joint_1']['max_position']}</param>
         </command_interface>
-        <state_interface name="position"/>
+        <state_interface name="position">
+          <param name="initial_value">${arm_initial_positions['joint_1']}</param>
+        </state_interface>
         <state_interface name="velocity"/>
         <state_interface name="effort"/>
@@ -23,5 +25,7 @@
           <param name="max">${arm_joint_limits['joint_2']['max_position']}</param>
         </command_interface>
-        <state_interface name="position"/>
+        <state_interface name="position">
+          <param name="initial_value">${arm_initial_positions['joint_2']}</param>
+        </state_interface>
         <state_interface name="velocity"/>
         <state_interface name="effort"/>
@@ -32,5 +36,7 @@
           <param name="max">${arm_joint_limits['joint_3']['max_position']}</param>
         </command_interface>
-        <state_interface name="position"/>
+        <state_interface name="position">
+          <param name="initial_value">${arm_initial_positions['joint_3']}</param>
+        </state_interface>
         <state_interface name="velocity"/>
         <state_interface name="effort"/>
@@ -41,5 +47,7 @@
           <param name="max">${arm_joint_limits['joint_4']['max_position']}</param>
         </command_interface>
-        <state_interface name="position"/>
+        <state_interface name="position">
+          <param name="initial_value">${arm_initial_positions['joint_4']}</param>
+        </state_interface>
         <state_interface name="velocity"/>
         <state_interface name="effort"/>
@@ -50,5 +58,7 @@
           <param name="max">${arm_joint_limits['joint_5']['max_position']}</param>
         </command_interface>
-        <state_interface name="position"/>
+        <state_interface name="position">
+          <param name="initial_value">${arm_initial_positions['joint_5']}</param>
+        </state_interface>
         <state_interface name="velocity"/>
         <state_interface name="effort"/>
@@ -59,5 +69,7 @@
           <param name="max">${arm_joint_limits['joint_6']['max_position']}</param>
         </command_interface>
-        <state_interface name="position"/>
+        <state_interface name="position">
+          <param name="initial_value">${arm_initial_positions['joint_6']}</param>
+        </state_interface>
         <state_interface name="velocity"/>
         <state_interface name="effort"/>

Commit message: fix(phase6): isolate drawing controller calibration

File: ros2_ws/src/abb_lab_gripper/urdf/irb1200_5_90_gz_gripper_control.urdf.xacro (robot description, xacro)
@@ -3,4 +3,5 @@
   <xacro:arg name="prefix" default=""/>
   <xacro:arg name="controller_config_file" default="$(find abb_lab_gripper)/config/irb1200_gripper_controllers.yaml"/>
+  <xacro:arg name="position_proportional_gain" default="1.0"/>
   <xacro:arg name="world_to_base_z" default="0"/>
   <!-- Keep the P3/P4 zero pose as the default.  Phase 5 passes a separate,
@@ -14,4 +15,5 @@
   <xacro:property name="prefix" value="$(arg prefix)"/>
   <xacro:property name="controller_config_file" value="$(arg controller_config_file)"/>
+  <xacro:property name="position_proportional_gain" value="$(arg position_proportional_gain)"/>
   <xacro:property name="world_to_base_z" value="$(arg world_to_base_z)"/>
   <xacro:property name="arm_joint_limits" value="${xacro.load_yaml('$(find abb_lab_description)/config/irb1200_5_90_control_limits.yaml')['joint_limits']}"/>
@@ -45,8 +47,8 @@
       <hold_joints>true</hold_joints>
       <!-- GazeboSimSystem maps a position error to joint velocity through this
-           documented proportional gain.  1.0 keeps the 40 mm finger stroke
-           below its 0.08 m/s hardware limit while reaching free-space action
-           goals before the controller's stall timeout. -->
-      <position_proportional_gain>1.0</position_proportional_gain>
+           documented proportional gain.  The default preserves the reviewed
+           P5 profile; Phase 6 supplies its separately tested simulation-only
+           gain through the exact spawned robot description. -->
+      <position_proportional_gain>${position_proportional_gain}</position_proportional_gain>
     </plugin>
   </gazebo>
